File: docs/thermostat-hardware/thermostat-hardware.kicad_sch (KiCad schematic)
At the start: 28 parts, among them J1 RELAY, J2 2.8_TFT_LCD, SW1 SW_Push, SW2 SW_Push, SW3 SW_Push, SW4 SW_Push, SW5 RotaryEncoder, SW6 SW_Push, SW7 SW_Push, U1 ESP32-C6-DevKitC-1, U2 DHT11, U3 IRM-H6xxT, U4 ESP32-DevKitC

Commit message: feat：增加ESP32-C6的管脚定义
Parts:
- added R12: 10k, Resistor_THT:R_Axial_DIN0207_L6.3mm_D2.5mm_P7.62mm_Horizontal, symbol Device:R
Connections:
- net +5V: now also R12.1
- net HEATER: now also U1.27 (GPIO22), R12.2; no longer U1.22 (GPIO9/BOOT)
Changed lines of the file:
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@@
 	)
 	(junction
+		(at 218.44 99.06)
+		(diameter 0)
+		(color 0 0 0 0)
+	)
+	(junction
 		(at 273.05 67.31)
 		(diameter 0)
@@
 	)
 	(junction
+		(at 228.6 85.09)
+		(diameter 0)
+		(color 0 0 0 0)
+	)
+	(junction
 		(at 134.62 38.1)
 		(diameter 0)
@@
 	(wire
 		(pts
+			(xy 232.41 99.06) (xy 232.41 90.17)
+		)
+		(stroke
+			(width 0)
+			(type default)
+		)
+	)
+	(wire
+		(pts
 			(xy 273.05 57.15) (xy 273.05 45.72)
 		)
@@
 	(wire
 		(pts
+			(xy 218.44 99.06) (xy 232.41 99.06)
+		)
+		(stroke
+			(width 0)
+			(type default)
+		)
+	)
+	(wire
+		(pts
 			(xy 123.19 170.18) (xy 123.19 167.64)
 		)
@@
 	(wire
 		(pts
+			(xy 218.44 87.63) (xy 218.44 85.09)
+		)
+		(stroke
+			(width 0)
+			(type default)
+		)
+	)
+	(wire
+		(pts
 			(xy 139.7 40.64) (xy 154.94 40.64)
 		)
@@
 	(wire
 		(pts
-			(xy 215.9 55.88) (xy 215.9 97.79)
+			(xy 270.51 77.47) (xy 273.05 77.47)
 		)
 		(stroke
@@
 	(wire
 		(pts
-			(xy 270.51 77.47) (xy 273.05 77.47)
+			(xy 152.4 24.13) (xy 152.4 30.48)
 		)
 		(stroke
@@
 	(wire
 		(pts
-			(xy 152.4 24.13) (xy 152.4 30.48)
+			(xy 233.68 142.24) (xy 196.85 142.24)
 		)
 		(stroke
@@
 	(wire
 		(pts
-			(xy 233.68 142.24) (xy 196.85 142.24)
+			(xy 82.55 175.26) (xy 82.55 172.72)
 		)
 		(stroke
@@
 	(wire
 		(pts
-			(xy 82.55 175.26) (xy 82.55 172.72)
+			(xy 152.4 30.48) (xy 154.94 30.48)
 		)
 		(stroke
@@
 	(wire
 		(pts
-			(xy 152.4 30.48) (xy 154.94 30.48)
+			(xy 115.57 127) (xy 233.68 127)
 		)
 		(stroke
@@
 	(wire
 		(pts
-			(xy 115.57 127) (xy 233.68 127)
+			(xy 214.63 43.18) (xy 214.63 99.06)
 		)
 		(stroke
@@
 	(wire
 		(pts
-			(xy 205.74 55.88) (xy 215.9 55.88)
-		)
-		(stroke
-			(width 0)
-			(type default)
-		)
-	)
-	(wire
-		(pts
 			(xy 110.49 36.83) (xy 110.49 66.04)
 		)
@@
 	(wire
 		(pts
+			(xy 218.44 85.09) (xy 228.6 85.09)
+		)
+		(stroke
+			(width 0)
+			(type default)
+		)
+	)
+	(wire
+		(pts
 			(xy 153.67 152.4) (xy 153.67 153.67)
 		)
@@
 	(wire
 		(pts
-			(xy 232.41 97.79) (xy 232.41 90.17)
-		)
-		(stroke
-			(width 0)
-			(type default)
-		)
-	)
-	(wire
-		(pts
 			(xy 125.73 43.18) (xy 125.73 55.88)
 		)
@@
 	(wire
 		(pts
+			(xy 218.44 95.25) (xy 218.44 99.06)
+		)
+		(stroke
+			(width 0)
+			(type default)
+		)
+	)
+	(wire
+		(pts
 			(xy 144.78 152.4) (xy 153.67 152.4)
 		)
@@
 	(wire
 		(pts
-			(xy 215.9 97.79) (xy 232.41 97.79)
+			(xy 214.63 99.06) (xy 218.44 99.06)
 		)
 		(stroke
@@
 	(wire
 		(pts
+			(xy 214.63 43.18) (xy 205.74 43.18)
+		)
+		(stroke
+			(width 0)
+			(type default)
+		)
+	)
+	(wire
+		(pts
 			(xy 260.35 67.31) (xy 227.33 67.31)
 		)
@@
 	)
 	(label "HEATER"
-		(at 217.17 97.79 0)
+		(at 224.79 99.06 0)
 		(effects
 			(font
@@
 	)
 	(symbol
+		(lib_id "Device:R")
+		(at 218.44 91.44 0)
+		(unit 1)
+		(body_style 1)
+		(exclude_from_sim no)
+		(in_bom yes)
+		(on_board yes)
+		(in_pos_files yes)
+		(dnp no)
+		(fields_autoplaced yes)
+		(property "Reference" "R12"
+			(at 220.98 90.1699 0)
+			(show_name no)
+			(do_not_autoplace no)
+			(effects
+				(font
+					(size 1.27 1.27)
+				)
+				(justify left)
+			)
+		)
+		(property "Value" "10k"
+			(at 220.98 92.7099 0)
+			(show_name no)
+			(do_not_autoplace no)
+			(effects
+				(font
+					(size 1.27 1.27)
+				)
+				(justify left)
+			)
+		)
+		(property "Footprint" "Resistor_THT:R_Axial_DIN0207_L6.3mm_D2.5mm_P7.62mm_Horizontal"
+			(at 216.662 91.44 90)
+			(hide yes)
+			(show_name no)
+			(do_not_autoplace no)
+			(effects
+				(font
+					(size 1.27 1.27)
+				)
+			)
+		)
+		(property "Datasheet" ""
+			(at 218.44 91.44 0)
+			(hide yes)
+			(show_name no)
+			(do_not_autoplace no)
+			(effects
+				(font
+					(size 1.27 1.27)
+				)
+			)
+		)
+		(property "Description" "Resistor"
+			(at 218.44 91.44 0)
+			(hide yes)
+			(show_name no)
+			(do_not_autoplace no)
+			(effects
+				(font
+					(size 1.27 1.27)
+				)
+			)
+		)
+		(pin "2"
+		)
+		(pin "1"
+		)
+		(instances
+			(project "thermostat-hardware"
+				(path "/3528b60d-1aad-4163-b1f0-ebe37a9f4906"
+					(reference "R12")
+					(unit 1)
+				)
+			)
+		)
+	)
+	(symbol
 		(lib_id "Connector:Conn_01x03_Pin")
 		(at 237.49 87.63 180)
@@
 		(in_pos_files yes)
 		(dnp no)
-		(fields_autoplaced yes)
 		(property "Reference" "#PWR09"
 			(at 228.6 96.52 0)
@@
 		)
 		(property "Value" "GND"
-			(at 228.6 95.25 0)
+			(at 228.854 93.98 0)
 			(show_name no)
 			(do_not_autoplace no)
